File: Rev A.sch (EAGLE design)
At the start: 19 parts, among them U1 LCD-16X28X2

Commit message: Did a lot of stuff
Parts:
- removed OPAMP: TLV2372IP, Texas Instruments_By_element14_Batch_1:TLV2372IP
- removed U1: LCD-16X28X2, SparkFun-Displays:LCD-16X28X2
- added 5VREG: 78L05SMD, linear:78L05SMD
- added C6, C9: 0.1uF, rcl:C-EUC0805
- added C7: 10uF, rcl:CPOL-EUE2.5-6
- added JP_BKL: (no value), pinhead:PINHD-2X2
- added LCD: LCD-16X28X2, SparkFun-Displays:LCD-16X28X2
- added OP1, OP2: TLV2372IP, Texas Instruments_By_element14_Batch_1:TLV2372IP
- added R8: 10kΩ, rcl:R-EU_R0805
- added RE1: ROTARTY_ENCODER, SparkFun-Electromechanical:ROTARTY_ENCODER
- added VO: 10kΩ, bourns:3386-G
- renumbered VREG to 3VREG
Connections:
- removed net N$2: C2.2, OPAMP.2IN-, R2.1
- new net +5V: 5VREGG$1.VOUT, C9.2, JP_BKL.4, LCD.VDD, VO.1
- new net CURR_SENSE: MCU.14, OP2.1IN-, OP2.1OUT
- new net DB4: LCD.DB4, MCU.11
- new net DB5: LCD.DB5, MCU.12
- new net DB6: LCD.DB6, MCU.13
- new net DB7: LCD.DB7, MCU.6
- new net LCD_EN: LCD.E, MCU.9
- new net N$1: C2.2, OP1.2IN-, OP2.1IN_+, R2.1
- new net N$10: LCD.VO, VO.2
- new net N$11: JP_BKL.3, LCD.A
- new net RE_A: MCU.7, RE1.A
- new net RE_B: MCU.15, RE1.B
- new net RE_BTN: MCU.5, R8.1, RE1.SW-
- new net RS: LCD.RS, MCU.8
- net CURR_SET: now also OP1.1IN-, OP1.1OUT, OP1.2IN+; no longer OPAMP.1IN-, OPAMP.1OUT, OPAMP.2IN+
- net GND: now also 5VREGG$1.GND@1, 5VREGG$1.GND@2, 5VREGG$1.GND@3, 5VREGG$1.GND@4, C6.1, C7.-, C9.1, LCD.K, LCD.R/W, LCD.VSS, OP1.GND, OP2.GND, RE1.C, RE1.SW+, VO.3; no longer OPAMP.GND, U1.K, U1.VSS
- net N$4: now also OP1.2OUT; no longer OPAMP.2OUT
- net N$6: now also 5VREGG$1.VIN
- net PWM_FILTERED: now also OP1.1IN_+; no longer OPAMP.1IN_+
- net VCC: now also C6.2, C7.+, OP1.VDD, OP2.VDD, R8.2; no longer OPAMP.VDD, U1.A, U1.VDD
Other:
- note added: "Maybe a JST?"
- note removed: "Add some filtering on the ouput?"
- note removed: "Maybe use more capacitance on the power rails to keep it quiet and operate well?"
- moved on the sheet: C1, C2, HEATSINK, N-CHANNEL, R2, R3, SHUNT

Commit message: Looks good to me
Parts:
- added 3V3, 5V, GND, IV, IVO, SGND: PTR1TP10SQ, testpad:PTR1TP10SQ
- added PWR_IN: M02JST-PTH-2, SparkFun-Connectors:M02JST-PTH-2
Connections:
- net +5V: now also 5V.TP
- net CURR_SENSE: now also IVO.TP
- net GND: now also GND.TP, PWR_IN.1, SGND.TP
- net N$13: now also IV.TP
- net TVIN: now also PWR_IN.2
- net VCC: now also 3V3.TP
Other:
- note removed: "Maybe a JST?"
- note removed: "Use block terminals for TVIN"
Changed lines of the file:
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@@
 <part name="C9" library="rcl" deviceset="C-EU" device="C0805" value="0.1uF"/>
 <part name="GND21" library="supply1" deviceset="GND" device=""/>
+<part name="PWR_IN" library="SparkFun-Connectors" deviceset="M02" device="JST-PTH-2"/>
+<part name="GND20" library="supply1" deviceset="GND" device=""/>
+<part name="3V3" library="testpad" deviceset="PTR1" device="TP10SQ"/>
+<part name="5V" library="testpad" deviceset="PTR1" device="TP10SQ"/>
+<part name="GND" library="testpad" deviceset="PTR1" device="TP10SQ"/>
+<part name="IV" library="testpad" deviceset="PTR1" device="TP10SQ"/>
+<part name="IVO" library="testpad" deviceset="PTR1" device="TP10SQ"/>
+<part name="SGND" library="testpad" deviceset="PTR1" device="TP10SQ"/>
 </parts>
 <sheets>
@@
 <plain>
 <text x="71.12" y="160.02" size="1.778" layer="91" rot="R90">Green 1206</text>
-<text x="212.09" y="22.86" size="3.81" layer="91">Use block terminals for TVIN</text>
 <text x="262.89" y="-5.08" size="1.778" layer="91" rot="R180">MTP3055</text>
-<text x="287.02" y="29.21" size="1.778" layer="91">Maybe a JST?</text>
 </plain>
 <instances>
@@
 <instance part="C9" gate="G$1" x="35.56" y="111.76" rot="R180"/>
 <instance part="GND21" gate="1" x="35.56" y="101.6"/>
+<instance part="PWR_IN" gate="G$1" x="279.4" y="22.86" rot="R180"/>
+<instance part="GND20" gate="1" x="269.24" y="5.08"/>
+<instance part="3V3" gate="G$1" x="50.8" y="172.72" rot="R90"/>
+<instance part="5V" gate="G$1" x="38.1" y="121.92" rot="R90"/>
+<instance part="GND" gate="G$1" x="-12.7" y="160.02" rot="R270"/>
+<instance part="IV" gate="G$1" x="267.97" y="-20.32" rot="R90"/>
+<instance part="IVO" gate="G$1" x="372.11" y="-58.42" rot="R90"/>
+<instance part="SGND" gate="G$1" x="267.97" y="-38.1" rot="R90"/>
 </instances>
 <busses>
@@
 <segment>
 <pinref part="SHUNT" gate="G$1" pin="1"/>
-<wire x1="265.43" y1="-35.56" x2="265.43" y2="-40.64" width="0.1524" layer="91"/>
+<wire x1="265.43" y1="-35.56" x2="265.43" y2="-38.1" width="0.1524" layer="91"/>
 <pinref part="GND3" gate="1" pin="GND"/>
+<pinref part="SGND" gate="G$1" pin="TP"/>
+<wire x1="265.43" y1="-38.1" x2="265.43" y2="-40.64" width="0.1524" layer="91"/>
+<junction x="265.43" y="-38.1"/>
 </segment>
 <segment>
 <pinref part="PWR" gate="G$1" pin="1"/>
 <wire x1="-15.24" y1="170.18" x2="-10.16" y2="170.18" width="0.1524" layer="91"/>
-<wire x1="-10.16" y1="170.18" x2="-10.16" y2="154.94" width="0.1524" layer="91"/>
+<wire x1="-10.16" y1="170.18" x2="-10.16" y2="160.02" width="0.1524" layer="91"/>
 <pinref part="GND4" gate="1" pin="GND"/>
+<pinref part="GND" gate="G$1" pin="TP"/>
+<wire x1="-10.16" y1="160.02" x2="-10.16" y2="154.94" width="0.1524" layer="91"/>
+<junction x="-10.16" y="160.02"/>
 </segment>
 <segment>
@@
 <wire x1="16.51" y1="102.87" x2="16.51" y2="96.52" width="0.1524" layer="91"/>
 <pinref part="GND17" gate="1" pin="GND"/>
+<junction x="16.51" y="102.87"/>
 </segment>
 <segment>
@@
 <wire x1="35.56" y1="109.22" x2="35.56" y2="104.14" width="0.1524" layer="91"/>
 <pinref part="GND21" gate="1" pin="GND"/>
+</segment>
+<segment>
+<pinref part="PWR_IN" gate="G$1" pin="1"/>
+<wire x1="271.78" y1="22.86" x2="269.24" y2="22.86" width="0.1524" layer="91"/>
+<wire x1="269.24" y1="22.86" x2="269.24" y2="7.62" width="0.1524" layer="91"/>
+<pinref part="GND20" gate="1" pin="GND"/>
 </segment>
 </net>
@@
 <pinref part="C7" gate="G$1" pin="+"/>
 <wire x1="43.18" y1="167.64" x2="43.18" y2="172.72" width="0.1524" layer="91"/>
+<pinref part="3V3" gate="G$1" pin="TP"/>
+<junction x="48.26" y="172.72"/>
 </segment>
 <segment>
@@
 <segment>
 <pinref part="N-CHANNEL" gate="G$1" pin="D"/>
-<wire x1="265.43" y1="-5.08" x2="265.43" y2="7.62" width="0.1524" layer="91"/>
-<label x="267.97" y="10.16" size="1.778" layer="95" rot="R180"/>
+<pinref part="PWR_IN" gate="G$1" pin="2"/>
+<wire x1="271.78" y1="20.32" x2="265.43" y2="20.32" width="0.1524" layer="91"/>
+<wire x1="265.43" y1="20.32" x2="265.43" y2="-5.08" width="0.1524" layer="91"/>
 </segment>
 </net>
@@
 <wire x1="369.57" y1="-58.42" x2="369.57" y2="-30.48" width="0.1524" layer="91"/>
 <junction x="369.57" y="-30.48"/>
+<pinref part="IVO" gate="G$1" pin="TP"/>
+<junction x="369.57" y="-58.42"/>
 </segment>
 <segment>
@@
 <pinref part="R2" gate="G$1" pin="2"/>
 <wire x1="255.27" y1="-20.32" x2="265.43" y2="-20.32" width="0.1524" layer="91"/>
+<pinref part="IV" gate="G$1" pin="TP"/>
 </segment>
 </net>
@@
 <wire x1="35.56" y1="116.84" x2="35.56" y2="121.92" width="0.1524" layer="91"/>
 <junction x="35.56" y="121.92"/>
-</segment>
-<segment>
+<pinref part="5V" gate="G$1" pin="TP"/>
+</segment>
+<segment>
